Commit message: added SLAM

File: description/robot.urdf.xacro (robot description, xacro)
@@ -2,8 +2,8 @@
 <robot xmlns:xacro="http://www.ros.org/wiki/xacro"  name="robot">
     <xacro:arg name="use_ros2_control" default="true"/>
-    <xacro:arg name="sim_mode" default="false"/>
     <xacro:include filename="robot_core.xacro" />
     <!-- <xacro:if value="$(arg use_ros2_control)"> -->
-        <xacro:include filename="ros2_control.xacro" />
+    <xacro:include filename="ros2_control.xacro" />
+    <!-- <xacro:include filename="lidar.xacro"/> -->
     <!-- </xacro:if> -->
     <!-- <xacro:unless value="$(arg use_ros2_control)">

File: description/robot_core.xacro (robot description, xacro)
@@ -17,4 +17,12 @@
     <link name="base_link">
     </link>
+    <!-- BASE FOOTPRINT LINK -->
+    <joint name="base_footprint_joint" type="fixed">
+        <parent link="base_link"/>
+        <child link="base_footprint"/>
+        <origin xyz="0 0 0" rpy="0 0 0"/>
+    </joint>
+    <link name="base_footprint">
+    </link>
     <!--CHASSIS LINK-->
     <joint name="chassis_joint" type="fixed">
@@ -202,3 +210,31 @@
         <material>Gazebo/Red</material>
     </gazebo>
+    <joint name = "laser_joint" type="fixed">
+        <parent link = "chassis"/>
+        <child link = "laser_frame"/>
+        <origin xyz = "0.1 0 0.175" rpy="0 0 0" />
+    </joint>
+    <link name = "laser_frame">
+        <visual>
+            <geometry>
+                <cylinder radius="0.05" length="0.04"/>
+            </geometry>
+            <material name="black"/>
+        </visual>
+        <visual>
+            <origin xyz="0 0 -0.05"/>
+            <geometry>
+                <cylinder radius="0.01" length="0.1"/>
+            </geometry>
+            <material name="black"/>
+        </visual>
+        <collision>
+            <geometry>
+                <cylinder radius="0.05" length="0.04"/>
+            </geometry>
+        </collision>
+        <xacro:inertial_cylinder mass="0.1" length="0.04" radius="0.05">
+            <origin xyz="0 0 0" rpy="0 0 0"/>
+        </xacro:inertial_cylinder>
+    </link>
 </robot>
