Commit message: Gazebo simulation

File: description/robot_core.xacro (robot description, xacro)
@@ -41,4 +41,7 @@
         </xacro:inertial_box>
     </link>
+    <gazebo reference="chassis">
+        <material>Gazebo/White</material>
+    </gazebo>
     <!-- LEFT WHEELS-->
     <!--Center wheel-->
@@ -65,4 +68,7 @@
         </xacro:inertial_cylinder>
     </link>
+    <gazebo reference="left_wheel">
+        <material>Gazebo/Red</material>
+    </gazebo>
     <!--front wheel-->
     <joint name="front_left_wheel_joint" type="continuous">
@@ -88,4 +94,7 @@
         </xacro:inertial_cylinder>
     </link>
+    <gazebo reference="front_left_wheel">
+        <material>Gazebo/Red</material>
+    </gazebo>
     <!--back wheel-->
     <joint name="back_left_wheel_joint" type="fixed">
@@ -111,4 +120,7 @@
         </xacro:inertial_cylinder>
     </link>
+    <gazebo reference="back_left_wheel">
+        <material>Gazebo/Red</material>
+    </gazebo>
     <!-- RIGHT WHEELS-->
     <!--Center wheel-->
@@ -135,4 +147,7 @@
         </xacro:inertial_cylinder>
     </link>
+    <gazebo reference="right_wheel">
+        <material>Gazebo/Red</material>
+    </gazebo>
     <!--Front wheel-->
     <joint name="front_right_wheel_joint" type="fixed">
@@ -158,4 +173,7 @@
         </xacro:inertial_cylinder>
     </link>
+    <gazebo reference="front_right_wheel">
+        <material>Gazebo/Red</material>
+    </gazebo>
     <!--back wheel-->
     <joint name="back_right_wheel_joint" type="continuous">
@@ -181,3 +199,6 @@
         </xacro:inertial_cylinder>
     </link>
+    <gazebo reference="back_right_wheel">
+        <material>Gazebo/Red</material>
+    </gazebo>
 </robot>

Commit message: cambio de topicos

File: description/robot_core.xacro (robot description, xacro)
@@ -238,3 +238,17 @@
         </xacro:inertial_cylinder>
     </link>
+    <link name="imu_link"/>
+    <joint
+        name="imu_joint"
+        type="fixed">
+        <origin
+        xyz="0.0 0 0.0"
+        rpy="0 -0.07 0" />
+        <parent
+        link="base_link" />
+        <child
+        link="imu_link" />
+        <axis
+        xyz="1 0 0" />
+    </joint>
 </robot>
